Commit message: Fix URDF: replace Unicode chars with ASCII to fix xacro XML parsing on Linux

File: src/jetson_bot_slam/urdf/jetson_bot.urdf.xacro (robot description, xacro)
@@ -4,5 +4,5 @@
   =====================
   Robot description for the mecanum-drive Jetson bot.
-  Physical dimensions (18.5 in wide × 13.5 in long, 4 in diameter wheels)
+  Physical dimensions (18.5 in wide x 13.5 in long, 4 in diameter wheels)
   -------------------------------------------------------------------------
   Base length (x) = 0.343 m  (13.5 in)
@@ -19,5 +19,5 @@
 -->
 <robot name="jetson_bot" xmlns:xacro="http://www.ros.org/wiki/xacro">
-  <!-- ── Colours ──────────────────────────────────────────────────────────── -->
+  <!-- Colours -->
   <material name="dark_grey">
     <color rgba="0.2 0.2 0.2 1"/>
@@ -32,5 +32,5 @@
     <color rgba="0.05 0.05 0.05 1"/>
   </material>
-  <!-- ── Properties ───────────────────────────────────────────────────────── -->
+  <!-- Properties -->
   <xacro:property name="base_length"    value="0.343"/>
   <xacro:property name="base_width"     value="0.470"/>
@@ -38,7 +38,7 @@
   <xacro:property name="wheel_radius"   value="0.0508"/>
   <xacro:property name="wheel_width"    value="0.038"/>
-  <xacro:property name="half_lx"        value="0.127"/>   <!-- half wheelbase -->
-  <xacro:property name="half_ly"        value="0.217"/>   <!-- half track     -->
-  <!-- ── Wheel macro ──────────────────────────────────────────────────────── -->
+  <xacro:property name="half_lx"        value="0.127"/>   <!-- half wheelbase (Lx) -->
+  <xacro:property name="half_ly"        value="0.217"/>   <!-- half track (Ly) -->
+  <!-- Wheel macro -->
   <xacro:macro name="wheel" params="name x y">
     <link name="${name}_link">

Commit message: Lidar Test + Frontier Exploration

File: src/jetson_bot_slam/urdf/jetson_bot.urdf.xacro (robot description, xacro)
@@ -4,15 +4,17 @@
   =====================
   Robot description for the mecanum-drive Jetson bot.
-  Physical dimensions (18.5 in wide x 13.5 in long, 4 in diameter wheels)
+  Physical dimensions (18.5 in wide x 13.5 in long, 13 in tall without LiDAR)
   Base length (x) = 0.343 m  (13.5 in)
   Base width  (y) = 0.470 m  (18.5 in)
-  Base height (z) = 0.080 m  (approx chassis height)
+  Base height (z) = 0.080 m  (approx chassis plate height)
   Wheel radius    = 0.0508 m (2 in)
   Wheel thickness = 0.038 m  (1.5 in)
   Half wheelbase  = 0.127 m  (5.0 in, Lx)
   Half track      = 0.217 m  (8.55 in, Ly)
+  Total height    = 0.330 m  (13 in, without LiDAR)
   Sensor placement:
   Camera:     USB camera mounted ~10 cm above base, at front-centre
-  Ultrasonic: HC-SR04 at front-centre, ~5 cm above base
+  LiDAR:      LDROBOT STL-27L, rear-right corner, 3.5 cm above chassis top
+  Ultrasonic: HC-SR04 rear-centre, facing backward, ~5 cm above base top
 -->
 <robot name="jetson_bot" xmlns:xacro="http://www.ros.org/wiki/xacro">
@@ -30,4 +32,7 @@
     <color rgba="0.05 0.05 0.05 1"/>
   </material>
+  <material name="green">
+    <color rgba="0.1 0.8 0.2 1"/>
+  </material>
   <!-- Properties -->
   <xacro:property name="base_length"    value="0.343"/>
@@ -38,4 +43,5 @@
   <xacro:property name="half_lx"        value="0.127"/>   <!-- half wheelbase (Lx) -->
   <xacro:property name="half_ly"        value="0.217"/>   <!-- half track (Ly) -->
+  <xacro:property name="lidar_height"   value="0.035"/>   <!-- 1.37 in above top plate -->
   <!-- Wheel macro -->
   <xacro:macro name="wheel" params="name x y">
@@ -130,5 +136,28 @@
   </joint>
   <!-- ===================================================================== -->
-  <!-- Ultrasonic sensor (HC-SR04, front-centre, ~5 cm above base top)       -->
+  <!-- LiDAR — LDROBOT STL-27L, rear-right corner, 3.5 cm above top plate   -->
+  <!-- ===================================================================== -->
+  <link name="lidar_link">
+    <visual>
+      <geometry><cylinder length="0.035" radius="0.035"/></geometry>
+      <material name="green"/>
+    </visual>
+  </link>
+  <joint name="lidar_joint" type="fixed">
+    <parent link="base_link"/>
+    <child  link="lidar_link"/>
+    <!-- Rear-right: -X (rear), -Y (right), above top plate -->
+    <origin xyz="${-base_length/2 + 0.06} ${-base_width/2 + 0.06} ${base_height/2 + lidar_height/2}"
+            rpy="0 0 0"/>
+  </joint>
+  <!-- laser_frame: the actual scan plane (required by ldlidar_stl_ros2) -->
+  <link name="laser_frame"/>
+  <joint name="laser_frame_joint" type="fixed">
+    <parent link="lidar_link"/>
+    <child  link="laser_frame"/>
+    <origin xyz="0 0 ${lidar_height/2}" rpy="0 0 0"/>
+  </joint>
+  <!-- ===================================================================== -->
+  <!-- Ultrasonic sensor (HC-SR04, REAR-centre, facing backward)             -->
   <!-- ===================================================================== -->
   <link name="ultrasonic_link">
@@ -141,6 +170,7 @@
     <parent link="base_link"/>
     <child  link="ultrasonic_link"/>
-    <origin xyz="${base_length/2 - 0.01} 0 ${base_height/2 + 0.05}"
-            rpy="0 0 0"/>
+    <!-- Rear-centre facing backward (rotated 180° around Z) -->
+    <origin xyz="${-base_length/2 + 0.01} 0 ${base_height/2 + 0.05}"
+            rpy="0 0 ${pi}"/>
   </joint>
 </robot>

Commit message: Xacro Fix + Collision Update

File: src/jetson_bot_slam/urdf/jetson_bot.urdf.xacro (robot description, xacro)
@@ -13,8 +13,8 @@
   Half track      = 0.217 m  (8.55 in, Ly)
   Total height    = 0.330 m  (13 in, without LiDAR)
-  Sensor placement:
-  Camera:     USB camera mounted ~10 cm above base, at front-centre
-  LiDAR:      LDROBOT STL-27L, rear-right corner, 3.5 cm above chassis top
-  Ultrasonic: HC-SR04 rear-centre, facing backward, ~5 cm above base top
+  Sensor placement (all centred widthwise, heights measured from ground):
+  LiDAR:      LDROBOT STL-27L, DEAD CENTRE of robot, scan plane at 14⅝"–15"
+  Camera:     USB camera at front-centre, sensor at 7⅝" height
+  Ultrasonic: HC-SR04 rear-centre, facing backward, at 6½" height
 -->
 <robot name="jetson_bot" xmlns:xacro="http://www.ros.org/wiki/xacro">
@@ -43,5 +43,9 @@
   <xacro:property name="half_lx"        value="0.127"/>   <!-- half wheelbase (Lx) -->
   <xacro:property name="half_ly"        value="0.217"/>   <!-- half track (Ly) -->
-  <xacro:property name="lidar_height"   value="0.035"/>   <!-- 1.37 in above top plate -->
+  <xacro:property name="lidar_height"   value="0.010"/>   <!-- spinning cylinder ~3/8 in -->
+  <!-- Ground-to-base_link offset: base_link is at centre of chassis plate,
+       chassis bottom sits at wheel-axle height (wheel_radius above ground) -->
+  <xacro:property name="base_z"  value="${wheel_radius + base_height/2}"/>
+  <!--  = 0.0508 + 0.040 = 0.0908 m above ground  -->
   <!-- Wheel macro -->
   <xacro:macro name="wheel" params="name x y">
@@ -64,6 +68,6 @@
       <parent link="base_link"/>
       <child  link="${name}_link"/>
-      <!-- wheels spin around Y axis; translate to corner positions, drop to ground -->
-      <origin xyz="${x} ${y} ${-base_height/2 + wheel_radius}"
+      <!-- Wheel axle is at the bottom of the chassis: z = -(base_height/2) -->
+      <origin xyz="${x} ${y} ${-base_height/2}"
               rpy="${pi/2} 0 0"/>
       <axis xyz="0 0 1"/>
@@ -77,5 +81,6 @@
     <parent link="base_footprint"/>
     <child  link="base_link"/>
-    <origin xyz="0 0 ${wheel_radius - base_height/2}"/>
+    <!-- base_link centre = wheel_radius + base_height/2 above ground -->
+    <origin xyz="0 0 ${base_z}"/>
   </joint>
   <!-- ===================================================================== -->
@@ -113,5 +118,5 @@
   <xacro:wheel name="wheel_BR" x="${-half_lx}" y="${-half_ly}"/>
   <!-- ===================================================================== -->
-  <!-- Camera link (USB camera, front-centre, ~10 cm above base top)         -->
+  <!-- Camera link (USB camera, front-centre, sensor at 7⅝" = 0.1937 m)    -->
   <!-- ===================================================================== -->
   <link name="camera_link">
@@ -124,6 +129,7 @@
     <parent link="base_link"/>
     <child  link="camera_link"/>
-    <!-- 14 cm forward, centre-left, 10 cm above base top -->
-    <origin xyz="${base_length/2 - 0.02} 0 ${base_height/2 + 0.10}"
+    <!-- Front-centre: x = base_length/2, y = 0
+         Height: 7.625" = 0.1937 m above ground → z relative to base_link -->
+    <origin xyz="${base_length/2} 0 ${0.1937 - base_z}"
             rpy="0 0 0"/>
   </joint>
@@ -136,9 +142,10 @@
   </joint>
   <!-- ===================================================================== -->
-  <!-- LiDAR — LDROBOT STL-27L, rear-right corner, 3.5 cm above top plate   -->
+  <!-- LiDAR — LDROBOT STL-27L, DEAD CENTRE of robot                        -->
+  <!-- Spinning bit: 14⅝" (0.3716 m) to 15" (0.381 m) above ground         -->
   <!-- ===================================================================== -->
   <link name="lidar_link">
     <visual>
-      <geometry><cylinder length="0.035" radius="0.035"/></geometry>
+      <geometry><cylinder length="${lidar_height}" radius="0.035"/></geometry>
       <material name="green"/>
     </visual>
@@ -147,9 +154,10 @@
     <parent link="base_link"/>
     <child  link="lidar_link"/>
-    <!-- Rear-right: -X (rear), -Y (right), above top plate -->
-    <origin xyz="${-base_length/2 + 0.06} ${-base_width/2 + 0.06} ${base_height/2 + lidar_height/2}"
+    <!-- Dead centre: x=0, y=0
+         LiDAR mid-height = (14.625+15)/2 = 14.8125" = 0.3763 m above ground -->
+    <origin xyz="0 0 ${0.3763 - base_z}"
             rpy="0 0 0"/>
   </joint>
-  <!-- laser_frame: the actual scan plane (required by ldlidar_stl_ros2) -->
+  <!-- laser_frame: the actual scan plane (top of spinning bit, required by ldlidar_stl_ros2) -->
   <link name="laser_frame"/>
   <joint name="laser_frame_joint" type="fixed">
@@ -160,4 +168,5 @@
   <!-- ===================================================================== -->
   <!-- Ultrasonic sensor (HC-SR04, REAR-centre, facing backward)             -->
+  <!-- Height: 6½" = 0.1651 m above ground                                   -->
   <!-- ===================================================================== -->
   <link name="ultrasonic_link">
@@ -170,6 +179,7 @@
     <parent link="base_link"/>
     <child  link="ultrasonic_link"/>
-    <!-- Rear-centre facing backward (rotated 180° around Z) -->
-    <origin xyz="${-base_length/2 + 0.01} 0 ${base_height/2 + 0.05}"
+    <!-- Rear-centre facing backward: x = -(base_length/2 - 0.01), y = 0
+         Height: 6.5" = 0.1651 m above ground → z relative to base_link -->
+    <origin xyz="${-(base_length/2 - 0.01)} 0 ${0.1651 - base_z}"
             rpy="0 0 ${pi}"/>
   </joint>
