Commit message: Add OVMM pipeline and scene graph navigation
Introduces a new end-to-end OVMM stack: topological map partitioning, SQLite scene graph storage, semantic waypoint dispatching, and a supervisor state machine that routes tasks from room navigation through visual docking and arm skill execution. Adds a unified `navigate_and_find` launch flow and wires new robot_control entry points for these nodes.

Also updates manipulation and platform integration details: dynamic target selection in `detection_node`, calibrated arm poses and hand-eye calibration path defaults, LiDAR UART defaults (`/dev/ttyTHS1`) across launch/compose/setup, and new scripts for LiDAR power control and arm vision lunge testing.

File: src/jetson_bot_slam/urdf/jetson_bot.urdf.xacro (robot description, xacro)
@@ -184,3 +184,17 @@
             rpy="0 0 ${pi}"/>
   </joint>
+  <!-- ===================================================================== -->
+  <!-- SO-ARM101 Arm Mount Base (Rear edge of chassis, facing rear)          -->
+  <!-- ===================================================================== -->
+  <link name="arm_base_link">
+    <visual>
+      <geometry><box size="0.080 0.080 0.040"/></geometry>
+      <material name="black"/>
+    </visual>
+  </link>
+  <joint name="arm_base_joint" type="fixed">
+    <parent link="base_link"/>
+    <child  link="arm_base_link"/>
+    <origin xyz="${-base_length/2} 0 0.040" rpy="0 0 ${pi}"/>
+  </joint>
 </robot>
